File: Load Cell Amp/Load Cell Amp R2.kicad_pcb (KiCad board)
At the start: 2 copper layers, 37 parts, among them J1 Conn_01x02_Male, J2 Conn_01x02_Male, J3 Conn_01x02_Male, J4 Conn_01x02_Male, J5 Conn_01x02_Male, J6 Conn_02x06_Odd_Even, J7 DB-26, U1 AD8227, U10 OP1177, U11 OP1177, U12 OP1177, U2 AD8227, U3 AD8227, U4 AD8227, U5 AD8227, U6 AD8227, U7 OP1177, U8 OP1177, U9 OP1177

Commit message: edits1
Parts:
- added C1: 100nF, Capacitors_SMD:C_0805, B.Cu at (128.9, 132.1)
- added C10: 100nF, Capacitors_SMD:C_0805, B.Cu at (143.3, 115.9)
- added C11: 100nF, Capacitors_SMD:C_0805, B.Cu at (143.3, 110.8)
- added C12: 100nF, Capacitors_SMD:C_0805, B.Cu at (143.3, 105.8)
- added C2: 100nF, Capacitors_SMD:C_0805, B.Cu at (128.9, 126.5)
- added C3: 100nF, Capacitors_SMD:C_0805, B.Cu at (128.9, 120.9)
- added C4: 100nF, Capacitors_SMD:C_0805, B.Cu at (128.9, 115.3)
- added C5: 100nF, Capacitors_SMD:C_0805, B.Cu at (129.2, 109.7)
- added C6: 100nF, Capacitors_SMD:C_0805, B.Cu at (129.2, 104.1)
- added C7: 100nF, Capacitors_SMD:C_0805, B.Cu at (143.3, 131.2)
- added C8: 100nF, Capacitors_SMD:C_0805, B.Cu at (143.3, 126.1)
- added C9: 100nF, Capacitors_SMD:C_0805, B.Cu at (143.3, 121.0)
- moved R1 2.54 mm to (123.8, 132.1)
- moved U1 2.54 mm to (128.9, 132.1)
- moved R2 2.03 mm to (123.8, 126.5)
- moved U2 2.03 mm to (128.9, 126.5)
- moved R3 1.52 mm to (123.8, 120.9)
- moved U3 1.52 mm to (128.9, 120.9)
- moved R4 1.02 mm to (123.8, 115.3)
- moved U4 1.02 mm to (128.9, 115.3)
- moved R5 0.51 mm to (123.8, 109.7)
- moved U5 0.51 mm to (128.9, 109.7)
Connections:
- U10 pad 3: Net-(R13-Pad2) -> Net-(R17-Pad2)
- U11 pad 3: Net-(R15-Pad2) -> Net-(R10-Pad1)
- U12 pad 3: Net-(R17-Pad2) -> Net-(R11-Pad2)
- U8 pad 3: Net-(R10-Pad1) -> Net-(R13-Pad2)
- U9 pad 3: Net-(R11-Pad2) -> Net-(R15-Pad2)
Routing:
- net +3V3: track 44.2 -> 91.6 mm
- net GND: track 77.3 -> 46.9 mm, vias 0 -> 12
- net SIG_0_-: track 51.1 -> 53.6 mm
- net VOUT_0: track 9.92 -> 7.38 mm
- net VOUT_2: track 21.7 -> 19.3 mm
- net SIG_0_+: track 41.9 -> 44.1 mm
- net REF4: track 32.1 -> 29.9 mm
- net VOUT_1: track 13.0 -> 10.9 mm
- net SIG_1_-: track 41.4 -> 43.5 mm
- net Net-(R11-Pad2): track 5.21 -> 7.30 mm
- net REF5: track 29.3 -> 27.2 mm
- net Net-(R17-Pad2): track 5.17 -> 3.11 mm
- net REF3: track 30.6 -> 28.6 mm
- net SIG_1_+: track 38.6 -> 40.3 mm
- net REF0: track 30.6 -> 29.1 mm
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Other:
- board outline added: 45.7 x 58.4 mm

Commit message: updates1.1
Connections:
- U10 pad 3: Net-(R17-Pad2) -> Net-(R13-Pad2)
- U11 pad 3: Net-(R10-Pad1) -> Net-(R15-Pad2)
- U12 pad 3: Net-(R11-Pad2) -> Net-(R17-Pad2)
- U8 pad 3: Net-(R13-Pad2) -> Net-(R10-Pad1)
- U9 pad 3: Net-(R15-Pad2) -> Net-(R11-Pad2)
Routing:
- net SIG_2_+: track 39.1 -> 24.3 mm
- net SIG_5_+: track 24.5 -> 37.1 mm
- net (no net): track 0.00 -> 2.25 mm
- net Net-(R11-Pad2): track 7.30 -> 5.21 mm
- net Net-(R17-Pad2): track 3.11 -> 5.17 mm
Changed lines of the file:
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@@
   (general
     (links 142)
-    (no_connects 92)
+    (no_connects 9)
     (area 114.249999 81.229999 160.070001 139.750001)
     (thickness 1.6)
@@
       (net 2 REF1))
     (pad 3 smd rect (at -2.2 0.325) (size 1.45 0.45) (layers F.Cu F.Paste F.Mask)
-      (net 44 "Net-(R13-Pad2)"))
+      (net 42 "Net-(R10-Pad1)"))
     (pad 4 smd rect (at -2.2 0.975) (size 1.45 0.45) (layers F.Cu F.Paste F.Mask)
       (net 15 GND))
@@
       (net 3 REF2))
     (pad 3 smd rect (at -2.2 0.325) (size 1.45 0.45) (layers F.Cu F.Paste F.Mask)
-      (net 45 "Net-(R15-Pad2)"))
+      (net 43 "Net-(R11-Pad2)"))
     (pad 4 smd rect (at -2.2 0.975) (size 1.45 0.45) (layers F.Cu F.Paste F.Mask)
       (net 15 GND))
@@
       (net 4 REF3))
     (pad 3 smd rect (at -2.2 0.325) (size 1.45 0.45) (layers F.Cu F.Paste F.Mask)
-      (net 46 "Net-(R17-Pad2)"))
+      (net 44 "Net-(R13-Pad2)"))
     (pad 4 smd rect (at -2.2 0.975) (size 1.45 0.45) (layers F.Cu F.Paste F.Mask)
       (net 15 GND))
@@
       (net 5 REF4))
     (pad 3 smd rect (at -2.2 0.325) (size 1.45 0.45) (layers F.Cu F.Paste F.Mask)
-      (net 42 "Net-(R10-Pad1)"))
+      (net 45 "Net-(R15-Pad2)"))
     (pad 4 smd rect (at -2.2 0.975) (size 1.45 0.45) (layers F.Cu F.Paste F.Mask)
       (net 15 GND))
@@
       (net 6 REF5))
     (pad 3 smd rect (at -2.2 0.325) (size 1.45 0.45) (layers F.Cu F.Paste F.Mask)
-      (net 43 "Net-(R11-Pad2)"))
+      (net 46 "Net-(R17-Pad2)"))
     (pad 4 smd rect (at -2.2 0.975) (size 1.45 0.45) (layers F.Cu F.Paste F.Mask)
       (net 15 GND))
@@
   (gr_arc (start 157.48 83.82) (end 157.48 81.28) (angle 90) (layer Edge.Cuts) (width 0.1))
   (gr_arc (start 116.844433 83.819996) (end 114.304433 83.819996) (angle 89.9) (layer Edge.Cuts) (width 0.1))
+  (segment (start 137.16 98.425) (end 137.16 97.0788) (width 0.1524) (layer F.Cu) (net 0))
+  (segment (start 136.51862 99.06638) (end 137.16 98.425) (width 0.1524) (layer F.Cu) (net 0))
   (segment (start 138.7856 130.175) (end 146.5834 130.175) (width 0.1524) (layer B.Cu) (net 1))
   (segment (start 146.5834 130.175) (end 146.8882 129.8702) (width 0.1524) (layer B.Cu) (net 1))
@@
   (segment (start 120.99615 115.432694) (end 120.99615 102.029773) (width 0.1524) (layer F.Cu) (net 26))
   (segment (start 120.99615 102.029773) (end 123.959543 99.06638) (width 0.1524) (layer F.Cu) (net 26))
-  (segment (start 123.959543 99.06638) (end 136.51862 99.06638) (width 0.1524) (layer F.Cu) (net 26))
-  (segment (start 137.16 98.425) (end 137.16 97.0788) (width 0.1524) (layer F.Cu) (net 26))
-  (segment (start 136.51862 99.06638) (end 137.16 98.425) (width 0.1524) (layer F.Cu) (net 26))
   (segment (start 126.205 111.633) (end 123.282838 111.633) (width 0.1524) (layer F.Cu) (net 27))
   (segment (start 139.176218 100.1522) (end 139.6492 99.679218) (width 0.1524) (layer F.Cu) (net 27))
@@
   (segment (start 139.05543 100.16177) (end 139.065 100.1522) (width 0.1524) (layer F.Cu) (net 27))
   (segment (start 139.6492 99.679218) (end 139.6492 98.7552) (width 0.1524) (layer F.Cu) (net 27))
+  (segment (start 112.718523 102.235) (end 125.2776 102.235) (width 0.1524) (layer F.Cu) (net 28))
   (segment (start 144.1704 100.3554) (end 144.1704 97.4344) (width 0.1524) (layer F.Cu) (net 28))
   (segment (start 143.3068 101.219) (end 144.1704 100.3554) (width 0.1524) (layer F.Cu) (net 28))
@@
   (segment (start 138.2014 123.5202) (end 138.7038 123.5202) (width 0.1524) (layer F.Cu) (net 42))
   (segment (start 138.7038 125.41) (end 138.2014 125.41) (width 0.1524) (layer F.Cu) (net 42))
-  (segment (start 141.0814 109.545) (end 138.9178 109.545) (width 0.1524) (layer F.Cu) (net 42))
   (segment (start 138.9126 123.729) (end 138.9126 124.7902) (width 0.1524) (layer F.Cu) (net 42))
   (segment (start 138.9126 124.7902) (end 138.9126 125.2012) (width 0.1524) (layer F.Cu) (net 42))
@@
   (segment (start 138.7038 123.5202) (end 138.9126 123.729) (width 0.1524) (layer F.Cu) (net 42))
   (segment (start 138.9126 125.2012) (end 138.7038 125.41) (width 0.1524) (layer F.Cu) (net 42))
+  (segment (start 141.0814 124.785) (end 138.9178 124.785) (width 0.1524) (layer F.Cu) (net 42))
   (segment (start 138.2014 118.46) (end 138.7038 118.46) (width 0.1524) (layer F.Cu) (net 43))
   (segment (start 138.7038 120.33) (end 138.2014 120.33) (width 0.1524) (layer F.Cu) (net 43))
-  (segment (start 138.9126 103.409) (end 138.9126 104.4702) (width 0.1524) (layer F.Cu) (net 43))
-  (segment (start 141.0814 104.465) (end 138.9178 104.465) (width 0.1524) (layer F.Cu) (net 43))
-  (segment (start 138.9126 104.4702) (end 138.9126 104.775) (width 0.1524) (layer F.Cu) (net 43))
-  (segment (start 138.9178 104.465) (end 138.9126 104.4702) (width 0.1524) (layer F.Cu) (net 43))
-  (segment (start 138.9126 104.775) (end 138.6332 105.0544) (width 0.1524) (layer F.Cu) (net 43))
-  (segment (start 138.7038 103.2002) (end 138.9126 103.409) (width 0.1524) (layer F.Cu) (net 43))
   (segment (start 138.938 118.6942) (end 138.938 119.7102) (width 0.1524) (layer F.Cu) (net 43))
   (segment (start 138.938 119.7102) (end 138.938 120.0958) (width 0.1524) (layer F.Cu) (net 43))
@@
   (segment (start 138.7038 118.46) (end 138.938 118.6942) (width 0.1524) (layer F.Cu) (net 43))
   (segment (start 138.938 120.0958) (end 138.7038 120.33) (width 0.1524) (layer F.Cu) (net 43))
-  (segment (start 141.0814 124.785) (end 138.9178 124.785) (width 0.1524) (layer F.Cu) (net 44))
+  (segment (start 141.0814 119.705) (end 138.9432 119.705) (width 0.1524) (layer F.Cu) (net 43))
   (segment (start 138.2014 113.35) (end 138.7038 113.35) (width 0.1524) (layer F.Cu) (net 44))
   (segment (start 138.7038 115.2398) (end 138.2014 115.2398) (width 0.1524) (layer F.Cu) (net 44))
@@
   (segment (start 138.7038 113.35) (end 138.9126 113.5588) (width 0.1524) (layer F.Cu) (net 44))
   (segment (start 138.9126 115.031) (end 138.7038 115.2398) (width 0.1524) (layer F.Cu) (net 44))
+  (segment (start 141.0814 114.625) (end 138.9178 114.625) (width 0.1524) (layer F.Cu) (net 44))
+  (segment (start 141.0814 109.545) (end 138.9178 109.545) (width 0.1524) (layer F.Cu) (net 45))
   (segment (start 138.9126 108.5088) (end 138.9126 109.9612) (width 0.1524) (layer F.Cu) (net 45))
-  (segment (start 141.0814 119.705) (end 138.9432 119.705) (width 0.1524) (layer F.Cu) (net 45))
   (segment (start 138.2014 108.3) (end 138.7038 108.3) (width 0.1524) (layer F.Cu) (net 45))
   (segment (start 138.9126 109.9612) (end 138.7038 110.17) (width 0.1524) (layer F.Cu) (net 45))
   (segment (start 138.7038 108.3) (end 138.9126 108.5088) (width 0.1524) (layer F.Cu) (net 45))
   (segment (start 138.7038 110.17) (end 138.2014 110.17) (width 0.1524) (layer F.Cu) (net 45))
-  (segment (start 141.0814 114.625) (end 138.9178 114.625) (width 0.1524) (layer F.Cu) (net 46))
+  (segment (start 138.9126 103.409) (end 138.9126 104.4702) (width 0.1524) (layer F.Cu) (net 46))
+  (segment (start 141.0814 104.465) (end 138.9178 104.465) (width 0.1524) (layer F.Cu) (net 46))
+  (segment (start 138.9126 104.4702) (end 138.9126 104.775) (width 0.1524) (layer F.Cu) (net 46))
+  (segment (start 138.9178 104.465) (end 138.9126 104.4702) (width 0.1524) (layer F.Cu) (net 46))
+  (segment (start 138.9126 104.775) (end 138.6332 105.0544) (width 0.1524) (layer F.Cu) (net 46))
+  (segment (start 138.7038 103.2002) (end 138.9126 103.409) (width 0.1524) (layer F.Cu) (net 46))
   (segment (start 138.6332 105.0544) (end 138.2268 105.0544) (width 0.1524) (layer F.Cu) (net 46))
   (segment (start 138.2268 105.0544) (end 138.2014 105.0798) (width 0.1524) (layer F.Cu) (net 46))

Commit message: edits1.2
Routing:
- net SIG_2_+: track 24.3 -> 39.0 mm
- net SIG_5_+: track 37.1 -> 24.5 mm
- net (no net): track 2.25 -> 0.00 mm
Changed lines of the file:
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@@
     (thickness 1.6)
     (drawings 8)
-    (tracks 523)
+    (tracks 525)
     (zones 0)
     (modules 49)
@@
   (gr_arc (start 157.48 83.82) (end 157.48 81.28) (angle 90) (layer Edge.Cuts) (width 0.1))
   (gr_arc (start 116.844433 83.819996) (end 114.304433 83.819996) (angle 89.9) (layer Edge.Cuts) (width 0.1))
-  (segment (start 137.16 98.425) (end 137.16 97.0788) (width 0.1524) (layer F.Cu) (net 0))
-  (segment (start 136.51862 99.06638) (end 137.16 98.425) (width 0.1524) (layer F.Cu) (net 0))
   (segment (start 138.7856 130.175) (end 146.5834 130.175) (width 0.1524) (layer B.Cu) (net 1))
   (segment (start 146.5834 130.175) (end 146.8882 129.8702) (width 0.1524) (layer B.Cu) (net 1))
@@
   (segment (start 119.93892 102.851027) (end 119.93892 101.591854) (width 0.1524) (layer F.Cu) (net 25))
   (segment (start 119.93892 101.591854) (end 123.521624 98.00915) (width 0.1524) (layer F.Cu) (net 25))
+  (segment (start 137.16 98.7044) (end 137.16 97.3836) (width 0.1524) (layer F.Cu) (net 26))
+  (segment (start 136.79802 99.06638) (end 137.16 98.7044) (width 0.1524) (layer F.Cu) (net 26))
+  (segment (start 136.69642 99.06638) (end 136.79802 99.06638) (width 0.1524) (layer F.Cu) (net 26))
+  (segment (start 136.11222 99.06638) (end 136.69642 99.06638) (width 0.1524) (layer F.Cu) (net 26))
+  (segment (start 123.959543 99.06638) (end 136.11222 99.06638) (width 0.1524) (layer F.Cu) (net 26))
   (segment (start 126.205 118.999) (end 124.562456 118.999) (width 0.1524) (layer F.Cu) (net 26))
   (segment (start 124.562456 118.999) (end 120.99615 115.432694) (width 0.1524) (layer F.Cu) (net 26))
@@
   (segment (start 139.05543 100.16177) (end 139.065 100.1522) (width 0.1524) (layer F.Cu) (net 27))
   (segment (start 139.6492 99.679218) (end 139.6492 98.7552) (width 0.1524) (layer F.Cu) (net 27))
-  (segment (start 112.718523 102.235) (end 125.2776 102.235) (width 0.1524) (layer F.Cu) (net 28))
   (segment (start 144.1704 100.3554) (end 144.1704 97.4344) (width 0.1524) (layer F.Cu) (net 28))
   (segment (start 143.3068 101.219) (end 144.1704 100.3554) (width 0.1524) (layer F.Cu) (net 28))
