File: Load Cell Amp/Load Cell Amp R2.kicad_pcb (KiCad board)
At the start: 2 copper layers, 45.7 x 58.4 mm, 49 parts, among them J1 Conn_01x02_Male, J2 Conn_01x02_Male, J3 Conn_01x02_Male, J4 Conn_01x02_Male, J5 Conn_01x02_Male, J6 Conn_02x06_Odd_Even, J7 DB-26, U1 AD8227, U10 OP1177, U11 OP1177, U12 OP1177, U2 AD8227, U3 AD8227, U4 AD8227, U5 AD8227, U6 AD8227, U7 OP1177, U8 OP1177, U9 OP1177

Commit message: Final changes
Routing:
- net GND: track 47.0 -> 57.6 mm
- net SIG_4_-: track 32.3 -> 40.4 mm, vias 0 -> 1
- net SIG_2_+: track 39.0 -> 46.9 mm
- net SIG_5_+: track 24.5 -> 32.1 mm
- net SIG_1_-: track 43.5 -> 49.9 mm
- net SIG_3_+: track 33.7 -> 40.0 mm
- net SIG_5_-: track 30.7 -> 35.0 mm, vias 0 -> 1
- net SIG_2_-: track 41.9 -> 45.3 mm
- net Net-(R15-Pad2): track 5.21 -> 6.81 mm
- net SIG_0_-: track 53.6 -> 54.4 mm
Other:
- board size 45.7 x 58.4 mm -> 45.7 x 59.2 mm
- net class Default: clearance 0.2 -> 0.1524; via_dia 0.6 -> 0.635; via_drill 0.4 -> 0.381
- rule trace_clearance: 0.2 -> 0.1524
- rule via_min_drill: 0.3 -> 0.381
- rule via_min_size: 0.4 -> 0.635
- board text added: "1 3 5 0 2 4"
- board text added: "3V3"
- board text added: "GND"
- board text added: "MASA AVIONICS LOADCELL AMP R2 - D. SALBERT - 11/3/2017"
- board text added: "VOUT"
